Commit message: feat: add a ros2 launch param to control whether to publish ros2 tf of odom
Add a ROS launch command parameter 'enable_odom_tf' to control whether to publish ros2 tf of odom.

Signed-off-by: weijshen <weijshen@qti.qualcomm.com>

File: qrb_ros_sim_gazebo/urdf/gazebo_qrb_mobile_manipulator_robot.urdf.xacro (robot description, xacro)
@@ -48,10 +48,12 @@
   <!-- Gazebo Plugins -->
   <!-- gz-sim-diff-drive-system controller -->
+  <xacro:arg name="enable_odom_tf" default="false"/>
+  <xacro:property name="tf_topic" value="${'tf' if '$(arg enable_odom_tf)' == 'true' else ''}" />
   <xacro:property name="separation_multiplier" value="1.15"/>
   <xacro:property name="radius_multiplier" value="1.0"/>
-  <xacro:property name="odom_update_rate" value="30"/>
+  <xacro:property name="odom_update_rate" value="50"/>
   <xacro:include filename="$(find qrb_ros_sim_gazebo)/urdf/xacro/gazebo_qrb_robot_base_diff_drive.xacro" />
   <xacro:qrb_robot_base_diff_drive ns="" wheel_separation="${wheel_separation}" separation_multiplier="${separation_multiplier}"
-      wheel_radius="${wheel_radius}" radius_multiplier="${radius_multiplier}" update_rate="${odom_update_rate}"/>
+      wheel_radius="${wheel_radius}" radius_multiplier="${radius_multiplier}" tf_topic="${tf_topic}" update_rate="${odom_update_rate}"/>
   <!-- gz-sim-joint-state-publisher-system controller -->
   <xacro:include filename="$(find qrb_ros_sim_gazebo)/urdf/xacro/gazebo_qrb_robot_base_joint_state_pub.xacro" />

File: qrb_ros_sim_gazebo/urdf/gazebo_qrb_robot_base.urdf.xacro (robot description, xacro)
@@ -25,4 +25,6 @@
   <!-- Gazebo Plugins -->
   <!-- gz-sim-diff-drive-system controller -->
+  <xacro:arg name="enable_odom_tf" default="false"/>
+  <xacro:property name="tf_topic" value="${'tf' if '$(arg enable_odom_tf)' == 'true' else ''}" />
   <xacro:property name="separation_multiplier" value="1.1525"/>
   <xacro:property name="radius_multiplier" value="1.0"/>
@@ -30,5 +32,5 @@
   <xacro:include filename="$(find qrb_ros_sim_gazebo)/urdf/xacro/gazebo_qrb_robot_base_diff_drive.xacro" />
   <xacro:qrb_robot_base_diff_drive ns="" wheel_separation="${wheel_separation}" separation_multiplier="${separation_multiplier}"
-      wheel_radius="${wheel_radius}" radius_multiplier="${radius_multiplier}" update_rate="${odom_update_rate}"/>
+      wheel_radius="${wheel_radius}" radius_multiplier="${radius_multiplier}" tf_topic="${tf_topic}" update_rate="${odom_update_rate}"/>
   <!-- gz-sim-joint-state-publisher-system controller -->
   <xacro:include filename="$(find qrb_ros_sim_gazebo)/urdf/xacro/gazebo_qrb_robot_base_joint_state_pub.xacro" />

File: qrb_ros_sim_gazebo/urdf/gazebo_qrb_robot_base_mini.urdf.xacro (robot description, xacro)
@@ -41,4 +41,6 @@
   <!-- Gazebo Plugins -->
   <!-- gz-sim-diff-drive-system controller -->
+  <xacro:arg name="enable_odom_tf" default="false"/>
+  <xacro:property name="tf_topic" value="${'tf' if '$(arg enable_odom_tf)' == 'true' else ''}" />
   <xacro:property name="separation_multiplier" value="1.125"/>
   <xacro:property name="radius_multiplier" value="1.0"/>
@@ -46,5 +48,5 @@
   <xacro:include filename="$(find qrb_ros_sim_gazebo)/urdf/xacro/gazebo_qrb_robot_base_diff_drive.xacro" />
   <xacro:qrb_robot_base_diff_drive ns="" wheel_separation="${wheel_separation}" separation_multiplier="${separation_multiplier}"
-      wheel_radius="${wheel_radius}" radius_multiplier="${radius_multiplier}" update_rate="${odom_update_rate}"/>
+      wheel_radius="${wheel_radius}" radius_multiplier="${radius_multiplier}" tf_topic="${tf_topic}" update_rate="${odom_update_rate}"/>
   <!-- gz-sim-joint-state-publisher-system controller -->
   <xacro:include filename="$(find qrb_ros_sim_gazebo)/urdf/xacro/gazebo_qrb_robot_base_joint_state_pub.xacro" />

File: qrb_ros_sim_gazebo/urdf/xacro/gazebo_qrb_robot_base_diff_drive.xacro (robot description, xacro)
@@ -2,5 +2,5 @@
 <robot xmlns:xacro="http://www.ros.org/wiki/xacro">
   <xacro:macro name="qrb_robot_base_diff_drive" params="ns:='' wheel_separation separation_multiplier:=1
-    wheel_radius radius_multiplier:=1 update_rate:=30 ">
+    wheel_radius radius_multiplier:=1 tf_topic:='' update_rate:=30 ">
     <xacro:property name="namespace" value="${ns + '/' if ns != '' else ''}" />
     <gazebo>
@@ -15,5 +15,5 @@
         <frame_id>${namespace}odom</frame_id>
         <child_frame_id>${namespace}base_footprint</child_frame_id>
-        <tf_topic>tf</tf_topic>
+        <tf_topic>${tf_topic}</tf_topic>
       </plugin>
     </gazebo>
