Commit message: update moveit demo.py
Signed-off-by: tengf <tengf@qti.qualcomm.com>

File: qrb_ros_moveit/config/rml_63.ros2_control.xacro (robot description, xacro)
@@ -7,4 +7,5 @@
                 <!-- By default, set up controllers for simulation. This won't work on real hardware -->
                 <plugin>mock_components/GenericSystem</plugin>
+                <!-- <plugin>gz_ros2_control/GazeboSimSystem</plugin> -->
             </hardware>
             <joint name="joint1">

File: qrb_ros_moveit/config/rml_63.urdf.xacro (robot description, xacro)
@@ -1,9 +1,45 @@
 <?xml version="1.0"?>
+<!-- Copyright (c) Qualcomm Technologies, Inc. and/or its subsidiaries.
+SPDX-License-Identifier: BSD-3-Clause-Clear -->
+<!-- <robot xmlns:xacro="http://www.ros.org/wiki/xacro" name="$(arg robot_name)"> -->
 <robot xmlns:xacro="http://www.ros.org/wiki/xacro" name="rml_63">
-    <xacro:arg name="initial_positions_file" default="initial_positions.yaml" />
-    <!-- Import rml_63 urdf file -->
-    <xacro:include filename="$(find qrb_ros_sim_gazebo)/urdf/gazebo_rml_63_gripper.urdf" />
-    <!-- Import control_xacro -->
-    <xacro:include filename="rml_63.ros2_control.xacro" />
-    <xacro:rml_63_ros2_control name="FakeSystem" initial_positions_file="$(arg initial_positions_file)"/>
+  <xacro:arg name="topic_ns" default=""/>
+  <!-- Import description urdf file -->
+  <xacro:include filename="$(find qrb_ros_sim_description)/urdf/rml_63_gripper_arm/rml_63.urdf" />
+  <xacro:include filename="$(find qrb_ros_sim_description)/urdf/rml_63_gripper_arm/gripper.urdf" />
+  <xacro:include filename="$(find qrb_ros_sim_description)/urdf/orbbec_cameras/gemini335_336.urdf.xacro" />
+  <xacro:rml_63 ns=""/>
+  <xacro:rml_gripper ns=""/>
+  <xacro:gemini_335_336 ns=""/>
+  <!-- Arm RGB camera -->
+  <xacro:arg name="enable_rgb_camera" default="false"/>
+  <xacro:arg name="rgb_camera_config" default=""/>
+  <xacro:if value="${'$(arg enable_rgb_camera)' if '$(arg rgb_camera_config)' != '' else 'false'}">
+    <xacro:include filename="$(find qrb_ros_sim_gazebo)/urdf/xacro/gazebo_rgb_camera.xacro" />
+    <xacro:gazebo_camera ns="" reference_link="camera_color_frame"
+      camera_params_yaml_path="$(arg rgb_camera_config)"/>
+  </xacro:if>
+  <!-- Arm Depth camera -->
+  <xacro:arg name="enable_depth_camera" default="false"/>
+  <xacro:arg name="depth_camera_config" default=""/>
+  <xacro:if value="${'$(arg enable_depth_camera)' if '$(arg depth_camera_config)' != '' else 'false'}">
+    <xacro:include filename="$(find qrb_ros_sim_gazebo)/urdf/xacro/gazebo_depth_camera.xacro" />
+    <xacro:gazebo_depth_camera ns="" reference_link="camera_depth_frame"
+      depth_camera_params_yaml_path="$(arg depth_camera_config)"/>
+  </xacro:if>
+  <joint name="arm_camera_joint" type="fixed">
+    <origin xyz="0.080 0 0.015" rpy="3.1415926 -1.570796 0"/>
+    <parent link="link6"/>
+    <child link="camera_link"/>
+  </joint>
+  <link name="world"/>
+  <joint name="arm_virtual_joint" type="fixed">
+    <parent link="world"/>
+    <child link="arm_base_link"/>
+  </joint>
+  <!-- ros2_control -->
+  <xacro:include filename="$(find qrb_ros_sim_gazebo)/urdf/xacro/rml_63_gripper_ros2_control.xacro" />
+  <xacro:rml_63_gripper_ros2_control ns="" topic_ns="$(arg topic_ns)"
+      initial_positions_yaml_path="$(find qrb_ros_sim_gazebo)/config/params/initial_positions.yaml"
+      ros2_controllers_yaml_path="$(find qrb_ros_sim_gazebo)/config/params/rml_63_ros2_controllers.yaml"/>
 </robot>
